File: Standalone/Flash.sch (KiCad schematic (older format))
At the start: 48 parts, among them CON1 GENESIS-CONN, J1 USB_B_Micro, U1 RT9193, U2 STM32F103C8Tx, U3 4069, U4 74HC590, U5 74LVC245, U6 74HC590, U7 74LVC245, U8 74HC590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

Commit message: Connected A22 and A23 on the cart connector for SNES support
Connections:
- net A21: now also CON1.B10 (A22)
- net A22: now also CON1.B11 (A23)
- no-connect marks 25 -> 23
Changed lines of the file:
@@
 NoConn ~ 14200 3600
 NoConn ~ 14200 3500
-NoConn ~ 14200 3400
-NoConn ~ 14200 3300
 NoConn ~ 14200 2600
 NoConn ~ 14200 2500
@@
 	1    0    0    -1
 $EndComp
+Text Label 14200 3300 0    50   ~ 0
+A21
+Text Label 14200 3400 0    50   ~ 0
+A22
 $EndSCHEMATC
